File: final/urd.kicad_pcb (KiCad board)
At the start: 2 copper layers, 100 x 55 mm, 83 parts, among them J2 Conn_01x04_Pin, J3 USB_C_Receptacle, Q1 IRF644PBF, Q10 MMBTA42, Q11 MMBTA42, Q12 MMBTA42, Q13 MMBTA42, Q2 MMBTA92, Q3 MMBTA42, Q4 MMBTA42, Q5 MMBTA42, Q6 MMBTA42, Q7 MMBTA42, Q8 MMBTA42, Q9 MMBTA42, U1 MAX1771ESA+T, U2 74HC595, U3 74HC595, U4 AMS1117-3.3, U5 STM32F103CBTx, U6 USBLC6-2SC6, U8 DS3231MZ, Y1 8Mhz

Commit message: Made PCB
Routed all traces and panelized different boards.
Parts:
- added H4: MountingHole, MountingHole:MountingHole_3.2mm_M3, F.Cu at (110.0, 100.5)
- added H5: MountingHole, MountingHole:MountingHole_3.2mm_M3, F.Cu at (0.00, 0.00)
- added H6: MountingHole, MountingHole:MountingHole_3.2mm_M3, F.Cu at (205.0, 0.00)
- added H7: MountingHole, MountingHole:MountingHole_3.2mm_M3, F.Cu at (0.00, 52.5)
- added H8: MountingHole, MountingHole:MountingHole_3.2mm_M3, F.Cu at (205.0, 52.5)
- added J1: Conn_01x05_Pin, Connector_PinHeader_2.54mm:PinHeader_1x05_P2.54mm_Vertical, F.Cu at (120.1, 80.5)
- added J4: Conn_01x10_Pin, Connector_IDC:IDC-Header_2x05_P2.54mm_Vertical, F.Cu at (103.2, 87.2)
- added J5: Conn_01x05_Pin, Connector_PinHeader_2.54mm:PinHeader_1x05_P2.54mm_Vertical, F.Cu at (60.5, 98.5)
- added J6: Conn_01x10_Pin, Connector_IDC:IDC-Header_2x05_P2.54mm_Vertical, B.Cu at (146.1, 45.5)
- added M1: ~, Custom:mouse-bite-5mm-slot, F.Cu at (5.00, 62.5)
- added M10: ~, Custom:mouse-bite-5mm-slot, F.Cu at (65.0, 105.5)
- added M11: ~, Custom:mouse-bite-5mm-slot, F.Cu at (105.0, 105.5)
- added M12: ~, Custom:mouse-bite-5mm-slot, F.Cu at (132.1, 89.5)
- added M13: ~, Custom:mouse-bite-5mm-slot, F.Cu at (170.2, 89.5)
- added M14: ~, Custom:mouse-bite-5mm-slot, F.Cu at (5.00, -10.0)
- added M15: ~, Custom:mouse-bite-5mm-slot, F.Cu at (200.0, -10.0)
- added M16: ~, Custom:mouse-bite-5mm-slot, F.Cu at (102.5, -10.0)
- added M17: ~, Custom:mouse-bite-5mm-slot, F.Cu at (132.1, 105.5)
- added M18: ~, Custom:mouse-bite-5mm-slot, F.Cu at (170.2, 105.5)
- added M4: ~, Custom:mouse-bite-5mm-slot, F.Cu at (85.0, 62.5)
- added M5: ~, Custom:mouse-bite-5mm-slot, F.Cu at (115.0, 75.4)
- added M6: ~, Custom:mouse-bite-5mm-slot, F.Cu at (132.1, 62.5)
- added M7: ~, Custom:mouse-bite-5mm-slot, F.Cu at (170.2, 62.5)
- added M8: ~, Custom:mouse-bite-5mm-slot, F.Cu at (5.00, 105.5)
- added M9: ~, Custom:mouse-bite-5mm-slot, F.Cu at (35.0, 105.5)
- added N2: ~, Custom:IN12, F.Cu at (40.9, 18.9)
- added N3: ~, Custom:IN12, F.Cu at (65.4, 18.9)
- added N4: ~, Custom:IN12, F.Cu at (89.9, 18.9)
- added N5: ~, Custom:IN12, F.Cu at (114.4, 18.9)
- added N6: ~, Custom:IN12, F.Cu at (138.9, 18.9)
- added N7: ~, Custom:IN12, F.Cu at (163.4, 18.9)
- added N8: ~, Custom:IN12, F.Cu at (187.9, 18.9)
- added Q14: MMBTA42, Package_TO_SOT_SMD:SOT-23, F.Cu at (3.00, 11.0)
- added Q15: MMBTA42, Package_TO_SOT_SMD:SOT-23, F.Cu at (3.00, 5.95)
- added Q16: MMBTA42, Package_TO_SOT_SMD:SOT-23, F.Cu at (201.3, 5.95)
- added Q17: MMBTA42, Package_TO_SOT_SMD:SOT-23, F.Cu at (201.3, 11.0)
- added Q18: MMBTA42, Package_TO_SOT_SMD:SOT-23, F.Cu at (201.3, 16.1)
- added Q19: MMBTA42, Package_TO_SOT_SMD:SOT-23, F.Cu at (201.3, 21.2)
- added Q20: MMBTA42, Package_TO_SOT_SMD:SOT-23, F.Cu at (3.00, 31.4)
- added R27: 10k, Resistor_SMD:R_0402_1005Metric, F.Cu at (61.4, 37.0)
- added R28: 10k, Resistor_SMD:R_0402_1005Metric, F.Cu at (85.9, 37.0)
- added R29: 10k, Resistor_SMD:R_0402_1005Metric, F.Cu at (110.4, 37.0)
- added R30: 10k, Resistor_SMD:R_0402_1005Metric, F.Cu at (134.9, 37.0)
- added R31: 10k, Resistor_SMD:R_0402_1005Metric, F.Cu at (159.4, 37.0)
- added R32: 10k, Resistor_SMD:R_0402_1005Metric, F.Cu at (183.9, 37.0)
- added R33: 10k, Resistor_SMD:R_1206_3216Metric, F.Cu at (21.4, 37.0)
- added R34: 10k, Resistor_SMD:R_1206_3216Metric, F.Cu at (45.9, 37.0)
- added R35: 10k, Resistor_SMD:R_1206_3216Metric, F.Cu at (70.4, 37.0)
- added R36: 10k, Resistor_SMD:R_1206_3216Metric, F.Cu at (94.9, 37.0)
- added R37: 10k, Resistor_SMD:R_1206_3216Metric, F.Cu at (119.4, 37.0)
- added R38: 10k, Resistor_SMD:R_1206_3216Metric, F.Cu at (143.9, 37.0)
- added R39: 10k, Resistor_SMD:R_1206_3216Metric, F.Cu at (168.4, 37.0)
- added R40: 10k, Resistor_SMD:R_1206_3216Metric, F.Cu at (192.9, 37.0)
- added R41: 10k, Resistor_SMD:R_0402_1005Metric, F.Cu at (204.3, 27.2)
- added R42: 10k, Resistor_SMD:R_0402_1005Metric, F.Cu at (0.00, 25.3)
- added R43: 10k, Resistor_SMD:R_0402_1005Metric, F.Cu at (0.00, 20.2)
- added R44: 10k, Resistor_SMD:R_0402_1005Metric, F.Cu at (155.0, 52.4)
- added R45: 10k, Resistor_SMD:R_0402_1005Metric, F.Cu at (0.00, 15.2)
- added R46: 10k, Resistor_SMD:R_0402_1005Metric, F.Cu at (0.00, 10.1)
- added R47: 10k, Resistor_SMD:R_0402_1005Metric, F.Cu at (0.00, 5.00)
- added R48: 10k, Resistor_SMD:R_0402_1005Metric, F.Cu at (204.3, 6.90)
- added R49: 10k, Resistor_SMD:R_0402_1005Metric, F.Cu at (204.3, 12.0)
- added R50: 10k, Resistor_SMD:R_0402_1005Metric, F.Cu at (204.3, 17.1)
- added R51: 10k, Resistor_SMD:R_0402_1005Metric, F.Cu at (204.3, 22.1)
- added R52: 10k, Resistor_SMD:R_0402_1005Metric, F.Cu at (0.00, 30.4)
- added R53: 100k, Resistor_SMD:R_1206_3216Metric, F.Cu at (2.99, 34.3)
- added SW1: SW_SPST, Button_Switch_Keyboard:SW_Cherry_MX_1.00u_PCB, F.Cu at (134.7, 70.3)
- added SW2: SW_SPST, Button_Switch_Keyboard:SW_Cherry_MX_1.00u_PCB, F.Cu at (153.7, 70.3)
- added SW3: SW_SPST, Button_Switch_Keyboard:SW_Cherry_MX_1.00u_PCB, F.Cu at (172.8, 70.3)
- added SW4: SW_SPST, Connector_PinHeader_2.54mm:PinHeader_1x02_P2.54mm_Vertical, F.Cu at (29.6, 95.5)
- added SW5: SW_SPST, Connector_PinHeader_2.54mm:PinHeader_1x02_P2.54mm_Vertical, F.Cu at (33.4, 95.5)
- added SW6: SW_SPST, Connector_PinHeader_2.54mm:PinHeader_1x02_P2.54mm_Vertical, F.Cu at (37.1, 95.5)
- added U7: 74HC595, Package_SO:SOIC-16_3.9x9.9mm_P1.27mm, F.Cu at (16.3, 47.0)
- C11: value 14p -> 100n
- C14: value 100n -> 10n
- C15: value 14p -> 1u
- C16: value 100n -> 1u
- C17: value 10n -> 22u; footprint Capacitor_SMD:C_0402_1005Metric -> Capacitor_SMD:C_0805_2012Metric
- C18: value 1u -> 22u; footprint Capacitor_SMD:C_0402_1005Metric -> Capacitor_SMD:C_0805_2012Metric
- C19: value 1u -> 100n
- C20: value 100n -> 14p
- C21: value 1n -> 14p
- C3: value 100n -> 100p/250v; footprint Capacitor_SMD:C_0402_1005Metric -> Capacitor_SMD:C_0805_2012Metric
- C5: value 100p/250v -> 100n/250v; footprint Capacitor_SMD:C_0805_2012Metric -> Capacitor_SMD:C_1206_3216Metric
- C6: value 100n/250v -> 100n; footprint Capacitor_SMD:C_1206_3216Metric -> Capacitor_SMD:C_0402_1005Metric
- C7: value 22u -> 100n; footprint Capacitor_SMD:C_0805_2012Metric -> Capacitor_SMD:C_0402_1005Metric
- C8: value 22u -> 1n; footprint Capacitor_SMD:C_0805_2012Metric -> Capacitor_SMD:C_0402_1005Metric
- J2: value Conn_01x04_Pin -> USB_C_Receptacle; footprint Connector_PinHeader_2.54mm:PinHeader_1x04_P2.54mm_Vertical -> Connector_USB:USB_C_Receptacle_HRO_TYPE-C-31-M-12
- J3: value USB_C_Receptacle -> Conn_01x04_Pin; footprint Connector_USB:USB_C_Receptacle_HRO_TYPE-C-31-M-12 -> Connector_PinHeader_2.54mm:PinHeader_1x04_P2.54mm_Vertical
- Q3, Q4, Q5, Q6, Q7, Q8, Q9: value MMBTA42 -> MMBTA92
- R10, R11: value 10k -> 5k1
- R12, R13, R6, R7: value 10k -> 1k5
- R15: value 100k -> 10k
- R16: footprint Resistor_SMD:R_1206_3216Metric -> Resistor_SMD:R_0402_1005Metric
- R18, R23: value 1k5 -> 100k
- R19, R20, R24: value 10k -> 100k
- R2: value 1M5 -> 10k; footprint Resistor_SMD:R_2512_6332Metric -> Resistor_SMD:R_0402_1005Metric
- R21, R22: value 5k1 -> 100k
- R25, R26: value 1k5 -> 10k
- R4: value 10k -> 1M5; footprint Resistor_SMD:R_0402_1005Metric -> Resistor_SMD:R_2512_6332Metric
- U2: value 74HC595 -> AMS1117-3.3; footprint Package_SO:SOIC-16_3.9x9.9mm_P1.27mm -> Package_TO_SOT_SMD:SOT-223-3_TabPin2
- U3: value 74HC595 -> DS3231MZ; footprint Package_SO:SOIC-16_3.9x9.9mm_P1.27mm -> Custom:SOP-8_4.93mmxP1.27mm
- U4: value AMS1117-3.3 -> USBLC6-2SC6; footprint Package_TO_SOT_SMD:SOT-223-3_TabPin2 -> Package_TO_SOT_SMD:SOT-23-6
- U6: value USBLC6-2SC6 -> 74HC595; footprint Package_TO_SOT_SMD:SOT-23-6 -> Package_SO:SOIC-16_3.9x9.9mm_P1.27mm
- U8: value DS3231MZ -> 74HC595; footprint Custom:SOP-8_4.93mmxP1.27mm -> Package_SO:SOIC-16_3.9x9.9mm_P1.27mm
- moved H3 255.2 mm to (0.00, 100.5)
- moved H1 253.6 mm to (0.00, 67.5)
- moved R25 235.1 mm to (12.4, 37.0), turned to -90 degrees
- moved R18 228.7 mm to (38.4, 37.0), turned to -90 degrees
- moved C3 227.0 mm to (9.10, 71.0)
- moved U1 217.6 mm to (23.1, 69.4)
- moved Q1 217.6 mm to (25.6, 73.9)
- moved C1 216.4 mm to (34.5, 73.6)
- moved L1 216.4 mm to (31.5, 84.9)
- moved C2 216.2 mm to (29.0, 69.5)
- moved D1 216.1 mm to (20.5, 84.9)
- moved RS1 215.5 mm to (16.6, 72.3)
- moved C4 214.2 mm to (15.8, 79.3)
- moved C6 213.8 mm to (18.8, 68.1), turned to -90 degrees
- moved R26 213.8 mm to (36.9, 37.0), turned to -90 degrees
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Connections:
- BT1 pad 2: GND -> GND1
- C1 pad 2: GND -> GND1
- C10 pad 1: /NRST -> +3V3_1
- C10 pad 2: GND -> GND1
- C11 pad 1: HSE_IN -> +3V3_1
- C11 pad 2: GND -> GND1
- C12 pad 1: +3.3V -> +3V3_1
- C12 pad 2: GND -> GND1
- C13 pad 1: +3.3V -> +3V3_1
- C13 pad 2: GND -> GND1
- C14 pad 1: +3.3V -> +3.3VA
- C14 pad 2: GND -> GND1
- C15 pad 1: HSE_OUT -> +3.3VA
- C15 pad 2: GND -> GND1
- C16 pad 1: +3.3V -> +3V3_1
- C16 pad 2: GND -> GND1
- C17 pad 1: +3.3VA -> VBUS
- C17 pad 2: GND -> GND1
- C18 pad 1: +3.3VA -> +3V3_1
- C18 pad 2: GND -> GND1
- C19 pad 1: +3.3V -> /NRST
- C19 pad 2: GND -> GND1
- C2 pad 2: GND -> GND1
- C20 pad 1: +3.3V -> HSE_IN
- C20 pad 2: GND -> GND1
- C21 pad 1: +BATT -> HSE_OUT
- C21 pad 2: GND -> GND1
- C3 pad 1: /REF_BYPASS -> FB
- C3 pad 2: GND -> 170V_1
- C4 pad 1: VCC -> 170V_1
- C4 pad 2: GND -> GND1
- C5 pad 1: FB -> 170V_1
- C5 pad 2: VCC -> GND1
- C6 pad 1: VCC -> /REF_BYPASS
- C6 pad 2: GND -> GND1
- C7 pad 1: VBUS -> +3V3_1
- C7 pad 2: GND -> GND1
- C8 pad 1: +3.3V -> +BATT
- C8 pad 2: GND -> GND1
- C9 pad 1: +3.3V -> +3V3_1
- C9 pad 2: GND -> GND1
- D1 pad 1: VCC -> 170V_1
- FB1 pad 2: +3.3V -> +3V3_1
- JP1 pad 1: +3.3V -> +3V3_1
- JP1 pad 2: /JMP_BOOT0 -> /PWR_LED_A
- JP2 pad 1: +3.3V -> +3V3_1
- JP2 pad 2: /PWR_LED_A -> /JMP_BOOT0
- N1 pad 1: /N1_CATHODE -> /N0_CATHODE
- Q10 pad 1: /S_7_BASE -> /S_0_BASE
- Q10 pad 2: GND -> GND2
- Q10 pad 3: NIXIE_7 -> NIXIE_0
- Q11 pad 1: /S_8_BASE -> /S_1_BASE
- Q11 pad 2: GND -> GND2
- Q11 pad 3: NIXIE_8 -> NIXIE_1
- Q12 pad 1: /S_DP_BASE -> /S_2_BASE
- Q12 pad 2: /DP_R -> GND2
- Q12 pad 3: NIXIE_DP -> NIXIE_2
- Q13 pad 1: /S_9_BASE -> /S_3_BASE
- Q13 pad 2: GND -> GND2
- Q13 pad 3: NIXIE_9 -> NIXIE_3
- Q2 pad 1: /N1_BASE -> /N0_BASE
- Q2 pad 2: VCC -> 170V_2
- Q2 pad 3: /N1_COLLECTOR -> /N0_COLLECTOR
- Q3 pad 1: /S_0_BASE -> /N1_BASE
- Q3 pad 2: GND -> 170V_2
- Q3 pad 3: NIXIE_0 -> /N1_COLLECTOR
- Q4 pad 1: /S_1_BASE -> /N2_BASE
- Q4 pad 2: GND -> 170V_2
- Q4 pad 3: NIXIE_1 -> /N2_COLLECTOR
- Q5 pad 1: /S_2_BASE -> /N3_BASE
- Q5 pad 2: GND -> 170V_2
- Q5 pad 3: NIXIE_2 -> /N3_COLLECTOR
- Q6 pad 1: /S_3_BASE -> /N4_BASE
- Q6 pad 2: GND -> 170V_2
- Q6 pad 3: NIXIE_3 -> /N4_COLLECTOR
- Q7 pad 1: /S_4_BASE -> /N5_BASE
- Q7 pad 2: GND -> 170V_2
- Q7 pad 3: NIXIE_4 -> /N5_COLLECTOR
- Q8 pad 1: /S_5_BASE -> /N6_BASE
- Q8 pad 2: GND -> 170V_2
- Q8 pad 3: NIXIE_5 -> /N6_COLLECTOR
- Q9 pad 1: /S_6_BASE -> /N7_BASE
- Q9 pad 2: GND -> 170V_2
- Q9 pad 3: NIXIE_6 -> /N7_COLLECTOR
- R1 pad 1: /FB_PD -> GND3
- R1 pad 2: GND -> HOUR_SW_D
- R10 pad 1: SIG_7 -> GND1
- R10 pad 2: /S_7_BASE -> USB_CC2
- R11 pad 1: SIG_8 -> GND1
- R11 pad 2: /S_8_BASE -> USB_CC1
- R12 pad 1: SIG_9 -> SCL
- R12 pad 2: /S_9_BASE -> +3V3_1
- R13 pad 1: SIG_DP -> SDA
- R13 pad 2: /S_DP_BASE -> +3V3_1
- R14 pad 1: /N1_BASE -> GND1
- R14 pad 2: N1_ENABLE -> POWER_SW
- R15 pad 1: /N1_BASE -> GND1
- R15 pad 2: VCC -> MODE_SW
- R16 pad 1: /N1_CATHODE -> GND1
- R16 pad 2: /N1_COLLECTOR -> ADJUST_SW
- R17 pad 1: /DP_R -> /N0_BASE
- R17 pad 2: GND -> 170V_2
- R18 pad 1: /PWR_LED_K -> /N1_BASE
- R18 pad 2: GND -> 170V_2
- R19 pad 1: GND -> /N2_BASE
- R19 pad 2: /JMP_BOOT0 -> 170V_2
- R2 pad 1: FB -> GND3
- R2 pad 2: VCC -> MINUTE_SW_D
- R20 pad 1: /BOOT0 -> /N3_BASE
- R20 pad 2: /JMP_BOOT0 -> 170V_2
- R21 pad 1: GND -> /N4_BASE
- R21 pad 2: USB_CC2 -> 170V_2
- R22 pad 1: GND -> /N5_BASE
- R22 pad 2: USB_CC1 -> 170V_2
- R23 pad 1: USB_D+ -> /N6_BASE
- R23 pad 2: +3.3V -> 170V_2
- R24 pad 1: SR_OE -> /N7_BASE
- R24 pad 2: +3.3V -> 170V_2
- R25 pad 1: SCL -> /N0_BASE
- R25 pad 2: +3.3V -> N0_ENABLE
- R26 pad 1: SDA -> /N1_BASE
- R26 pad 2: +3.3V -> N1_ENABLE
- R3 pad 1: SIG_0 -> GND3
- R3 pad 2: /S_0_BASE -> SECOND_SW_D
- R4 pad 1: SIG_1 -> FB
- R4 pad 2: /S_1_BASE -> 170V_1
- R5 pad 1: SIG_2 -> /FB_PD
- R5 pad 2: /S_2_BASE -> GND1
- R6 pad 1: SIG_3 -> /PWR_LED_K
- R6 pad 2: /S_3_BASE -> GND1
- R7 pad 1: SIG_4 -> USB_D+
- R7 pad 2: /S_4_BASE -> +3V3_1
- R8 pad 1: SIG_5 -> /BOOT0
- R8 pad 2: /S_5_BASE -> /JMP_BOOT0
- R9 pad 1: SIG_6 -> GND1
- R9 pad 2: /S_6_BASE -> /JMP_BOOT0
- RS1 pad 2: GND -> GND1
- U1 pad 4: GND -> GND1
- U1 pad 6: GND -> GND1
- U1 pad 7: GND -> GND1
- U2 pad 1: SIG_5 -> GND1
- U2 pad 2: SIG_6 -> +3V3_1
- U2 pad 3: SIG_7 -> VBUS
- U3 pad 1: SIG_2 -> unconnected-(U3-32KHZ-Pad1)
- U3 pad 2: SIG_3 -> +BATT
- U3 pad 4: unconnected-(U3-QE-Pad4) -> +3V3_1
- U3 pad 5: unconnected-(U3-QF-Pad5) -> GND1
- U3 pad 6: unconnected-(U3-QG-Pad6) -> +3V3_1
- U3 pad 7: unconnected-(U3-QH-Pad7) -> SDA
- U3 pad 8: GND -> SCL
- U4 pad 1: GND -> /CONN_D-
- U4 pad 2: +3.3V -> GND1
- U4 pad 3: VBUS -> /CONN_D+
- U5 pad 1: +3.3V -> +3V3_1
- U5 pad 14: SR_LATCH -> DIG_SR_LATCH_H
- U5 pad 15: SR_CLK -> DIG_SR_CLK_H
- U5 pad 16: SR_OE -> unconnected-(U5-PA6-Pad16)
- U5 pad 17: SR_DATA -> DIG_SR_DATA_H
- U5 pad 18: N1_ENABLE -> unconnected-(U5-PB0-Pad18)
- U5 pad 19: unconnected-(U5-PB1-Pad19) -> SR_OE_H
- U5 pad 23: GND -> GND1
- U5 pad 24: +3.3V -> +3V3_1
- U5 pad 25: unconnected-(U5-PB12-Pad25) -> NIX_SR_LATCH_H
- U5 pad 26: unconnected-(U5-PB13-Pad26) -> NIX_SR_CLK_H
- U5 pad 28: unconnected-(U5-PB15-Pad28) -> NIX_SR_DATA_H
- U5 pad 35: GND -> GND1
- U5 pad 36: +3.3V -> +3V3_1
- U5 pad 38: unconnected-(U5-PA15-Pad38) -> POWER_SW
- U5 pad 39: unconnected-(U5-PB3-Pad39) -> MODE_SW
- U5 pad 40: unconnected-(U5-PB4-Pad40) -> ADJUST_SW
- U5 pad 41: unconnected-(U5-PB5-Pad41) -> HOUR_SW_H
- U5 pad 42: unconnected-(U5-PB6-Pad42) -> MINUTE_SW_H
- U5 pad 43: unconnected-(U5-PB7-Pad43) -> SECOND_SW_H
- U5 pad 47: GND -> GND1
- U5 pad 48: +3.3V -> +3V3_1
- U5 pad 8: GND -> GND1
- U6 pad 1: /CONN_D- -> unconnected-(U6-QB-Pad1)
- U6 pad 2: GND -> unconnected-(U6-QC-Pad2)
- U6 pad 3: /CONN_D+ -> SIG_6
- U6 pad 4: USB_D+ -> SIG_7
- U6 pad 5: VBUS -> SIG_8
- U6 pad 6: USB_D- -> SIG_9
- U8 pad 1: unconnected-(U8-32KHZ-Pad1) -> N3_ENABLE
- U8 pad 2: +BATT -> N2_ENABLE
- U8 pad 3: unconnected-(U8-~{INT}/SQW-Pad3) -> N1_ENABLE
- U8 pad 4: +3.3V -> N0_ENABLE
- U8 pad 5: GND -> N4_ENABLE
- U8 pad 6: +3.3V -> N5_ENABLE
- U8 pad 7: SDA -> N6_ENABLE
- U8 pad 8: SCL -> GND2
- Y1 pad 2: GND -> GND1
- Y1 pad 4: GND -> GND1
Routing:
- net 170V_2: track 0.00 -> 520.8 mm
- net +3V3_2: track 0.00 -> 251.9 mm, vias 0 -> 3
- net +3V3_1: track 0.00 -> 244.8 mm, vias 0 -> 3
- net NIXIE_7: track 9.89 -> 203.9 mm
- net +3.3V: track 193.4 -> 0.00 mm, vias 4 -> 0
- net DIG_SR_CLK_D: track 0.00 -> 191.4 mm, vias 0 -> 2
- net NIXIE_DP: track 13.7 -> 204.6 mm, vias 1 -> 0
- net DIG_SR_CHAIN: track 0.00 -> 190.4 mm, vias 0 -> 4
- net NIXIE_9: track 7.74 -> 194.6 mm
- net NIXIE_6: track 14.0 -> 199.7 mm
- net NIXIE_1: track 20.4 -> 205.5 mm, vias 1 -> 0
- net NIXIE_0: track 7.35 -> 190.7 mm
- net SR_OE_D: track 0.00 -> 183.3 mm, vias 0 -> 2
- net NIXIE_8: track 8.14 -> 190.4 mm
- net DIG_SR_LATCH_D: track 0.00 -> 180.0 mm, vias 0 -> 2
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- added copper zone on F.Cu, net +3V3_1
- added copper zone on F.Cu, net 170V_1
- added copper zone on B.Cu, net GND1
- added copper zone on F.Cu, net GND1
- added copper zone on B.Cu, net GND2
- added copper zone on B.Cu, net GND3
- removed copper zone on F.Cu, net +3.3V
- removed copper zone on F.Cu, net /N1_BASE
- removed copper zone on B.Cu, net GND
- removed copper zone on F.Cu, net GND
- removed copper zone on F.Cu, net VCC
Other:
- board size 100 x 55 mm -> 220 x 130.5 mm
- board text removed: "+"
- board text removed: "-"
- board text removed: "- CLK DIO +"
- board text removed: "LWQ"
