File: final/urd.kicad_sch (KiCad schematic)
At the start: 135 parts, among them J1 Conn_01x10_Pin, J2 Conn_01x04_Pin, J3 USB_C_Receptacle, J4 Conn_01x10_Pin, J5 Conn_01x06_Pin, J6 Conn_01x06_Pin, Q1 IRF644PBF, Q10 MMBTA42, Q11 MMBTA42, Q12 MMBTA42, Q14 MMBTA92, Q15 MMBTA92, Q16 MMBTA92, Q17 MMBTA92, Q18 MMBTA92, Q19 MMBTA92, Q2 MMBTA42, Q20 MMBTA92, Q21 MMBTA92, Q3 MMBTA42, Q4 MMBTA42, Q5 MMBTA42, Q6 MMBTA42, Q7 MMBTA42, Q8 MMBTA42, Q9 MMBTA42, SW1 SW_SPST, SW2 SW_SPST, SW3 SW_SPST, SW4 SW_SPST, SW5 SW_SPST, SW6 SW_SPST, U1 MAX1771ESA+T, U2 74HC595, U3 74HC595, U4 AMS1117-3.3, U5 STM32F103CBTx, U6 USBLC6-2SC6, U7 74HC595, U8 DS3231MZ, Y1 8Mhz

Commit message: Made PCB
Routed all traces and panelized different boards.
Parts:
- removed J5, J6: Conn_01x06_Pin, Connector_IDC:IDC-Header_2x03_P2.54mm_Vertical, symbol Connector:Conn_01x06_Pin
- removed JP2: SolderJumper_2_Open, Connector_PinHeader_2.54mm:PinHeader_1x02_P2.54mm_Vertical, symbol Jumper:SolderJumper_2_Open
- added H4, H5, H6, H7, H8: MountingHole, MountingHole:MountingHole_3.2mm_M3, symbol Mechanical:MountingHole
- added J1, J5: Conn_01x05_Pin, Connector_PinHeader_2.54mm:PinHeader_1x05_P2.54mm_Vertical, symbol Connector:Conn_01x05_Pin
- added JP1: SolderJumper_2_Open, Connector_PinHeader_2.54mm:PinHeader_1x02_P2.54mm_Vertical, symbol Jumper:SolderJumper_2_Open
- added M1, M10, M11, M12, M13, M14, M15, M16, M17, M18, M2, M3, M4, M5, M6, M7, M8, M9: ~, Custom:mouse-bite-5mm-slot, symbol Custom:Mouse_Bite
- R53: renamed from R11; footprint Resistor_SMD:R_0402_1005Metric -> Resistor_SMD:R_1206_3216Metric
- renumbered C12 to C10, C13 to C11, C14 to C12, C16 to C13, C17 to C14, C18 to C15, C19 to C16, C7 to C17, C8 to C18, C10 to C19, C11 to C20, C15 to C21, C5 to C3, C6 to C5, C3 to C6, C20 to C7, C21 to C8, J3 to J2, J2 to J3, J1 to J6, JP1 to JP2, N2 to N1, N3 to N2, N4 to N3, N5 to N4, N6 to N5, N7 to N6, N8 to N7, N9 to N8, Q2 to Q10, Q6 to Q11, Q10 to Q12, Q3 to Q13, Q7 to Q14, Q11 to Q15, Q4 to Q16, Q8 to Q17, Q12 to Q18, Q5 to Q19, Q14 to Q2, Q9 to Q20, Q15 to Q3, Q16 to Q4, Q17 to Q5, Q18 to Q6, Q19 to Q7, Q20 to Q8, Q21 to Q9, R51 to R1, R21 to R10, R22 to R11, R25 to R12, R26 to R13, R16 to R14, R17 to R15, R24 to R16, R28 to R17, R31 to R18, R34 to R19, R52 to R2, R37 to R20, R40 to R21, R43 to R22, R46 to R23, R49 to R24, R29 to R25, R32 to R26, R35 to R27, R38 to R28, R41 to R29, R53 to R3, R44 to R30, R47 to R31, R50 to R32, R27 to R33, R30 to R34, R33 to R35, R39 to R37, R42 to R38, R45 to R39, R2 to R4, R48 to R40, R3 to R41, R7 to R42, R12 to R43, R15 to R44, R4 to R45, R8 to R46, R13 to R47, R5 to R48, R9 to R49, R1 to R5, R14 to R50, R6 to R51, R10 to R52, R18 to R6, R23 to R7, R20 to R8, R19 to R9, SW4 to SW1, SW5 to SW2, SW6 to SW3, SW1 to SW4, SW2 to SW5, SW3 to SW6, U4 to U2, U8 to U3, U6 to U4, U2 to U6, U3 to U7, U7 to U8
Connections:
- net HOUR_SW is gone; now on net HOUR_SW_D: R1.2, SW1.2 (B)
- net MINUTE_SW is gone; now on net MINUTE_SW_D: R2.2, SW2.2 (B)
- net SECOND_SW is gone; now on net SECOND_SW_D: R3.2, SW3.2 (B)
- net SR_OE is gone; now on net SR_OE_D: R44.1, U6.13 (~{OE}), U7.13 (~{OE}), U8.13 (~{OE})
- net ADJUST_SW: now also U5.40 (PB4)
- net DIG_SR_CLK_H: now also J4.3 (Pin_3); no longer J4.6 (Pin_6)
- net DIG_SR_DATA_H: now also J4.4 (Pin_4); no longer J4.5 (Pin_5)
- net DIG_SR_LATCH_H: now also J4.2 (Pin_2); no longer J4.7 (Pin_7)
- net HOUR_SW_D: now also J1.4 (Pin_4)
- net HOUR_SW_H: now also U5.41 (PB5), J5.4 (Pin_4)
- net MINUTE_SW_D: now also J1.3 (Pin_3)
- net MINUTE_SW_H: now also U5.42 (PB6), J5.3 (Pin_3)
- net MODE_SW: now also U5.39 (PB3)
- net N0_ENABLE: now also U8.4 (QE); no longer U8.15 (QA)
- net N1_ENABLE: now also U8.3 (QD); no longer U8.1 (QB)
- net N3_ENABLE: now also U8.1 (QB); no longer U8.3 (QD)
- net N4_ENABLE: now also U8.5 (QF); no longer U8.4 (QE)
- net N5_ENABLE: now also U8.6 (QG); no longer U8.5 (QF)
- net N6_ENABLE: now also U8.7 (QH); no longer U8.6 (QG)
- net N7_ENABLE: now also U8.15 (QA); no longer U8.7 (QH)
- net NIX_SR_CLK_H: now also J4.7 (Pin_7); no longer J4.3 (Pin_3)
- net NIX_SR_DATA_H: now also J4.8 (Pin_8); no longer J4.2 (Pin_2)
- net NIX_SR_LATCH_H: now also J4.6 (Pin_6); no longer J4.4 (Pin_4)
- net POWER_SW: now also U5.38 (PA15)
- net PWR_LED_A: now also JP1.2 (B)
- net SECOND_SW_D: now also J1.2 (Pin_2)
- net SECOND_SW_H: now also U5.43 (PB7), J5.2 (Pin_2)
- net SIG_0: now also U6.7 (QH); no longer U6.6 (QG)
- net SIG_1: now also U7.2 (QC); no longer U7.15 (QA)
- net SIG_2: now also U7.3 (QD); no longer U7.1 (QB)
- net SIG_3: now also U7.4 (QE); no longer U7.2 (QC)
- net SIG_4: now also U7.5 (QF); no longer U6.15 (QA)
- net SIG_5: now also U7.6 (QG); no longer U6.1 (QB)
- net SIG_6: now also U6.3 (QD); no longer U6.2 (QC)
- net SIG_7: now also U6.4 (QE); no longer U6.3 (QD)
- net SIG_8: now also U6.5 (QF); no longer U6.4 (QE)
- net SIG_9: now also U6.6 (QG); no longer U6.5 (QF)
- net SIG_DP: now also U7.1 (QB); no longer U6.7 (QH)
- net SR_OE_H: now also J4.5 (Pin_5), U5.19 (PB1); no longer J4.8 (Pin_8)
- net +3.3V renamed +3V3_1
- net +3V3_1: now also J5.5 (Pin_5), JP1.1 (A); no longer J6.9 (Pin_9), R44.2, SW1.1 (A), SW2.1 (A), SW3.1 (A), U6.10 (~{SRCLR}), U6.16 (VCC), U7.10 (~{SRCLR}), U7.16 (VCC), U8.10 (~{SRCLR}), U8.16 (VCC)
- net GND renamed GND1
- net GND1: now also J5.1 (Pin_1); no longer J6.1 (Pin_1), Q10.2 (E), Q11.2 (E), Q12.2 (E), Q13.2 (E), Q14.2 (E), Q15.2 (E), Q16.2 (E), Q17.2 (E), Q18.2 (E), Q19.2 (E), R1.1, R2.1, R3.1, R53.2, U6.8 (GND), U7.8 (GND), U8.8 (GND)
- net VCC renamed 170V_2
- net 170V_2: now also J6.9 (Pin_9); no longer C3.2, C4.1, C5.1, D1.1 (K), J4.10 (Pin_10), J6.10 (Pin_10), R4.2
- new net +3V3_2: J6.10 (Pin_10), R44.2, U6.10 (~{SRCLR}), U6.16 (VCC), U7.10 (~{SRCLR}), U7.16 (VCC), U8.10 (~{SRCLR}), U8.16 (VCC)
- new net +3V3_3: J1.5 (Pin_5), SW1.1 (A), SW2.1 (A), SW3.1 (A)
- new net 170V_1: C3.2, C4.1, C5.1, D1.1 (K), J4.10 (Pin_10), R4.2
- new net GND2: J6.1 (Pin_1), Q10.2 (E), Q11.2 (E), Q12.2 (E), Q13.2 (E), Q14.2 (E), Q15.2 (E), Q16.2 (E), Q17.2 (E), Q18.2 (E), Q19.2 (E), R53.2, U6.8 (GND), U7.8 (GND), U8.8 (GND)
- new net GND3: J1.1 (Pin_1), R1.1, R2.1, R3.1
- no-connect marks 50 -> 34
Other:
- note added: "For KiCad ERC"
- note added: "Mounting Holes"
- note added: "Mouse Bites"
- note added: "Vout = Vref((R2 / R1) + 1) Vref = 1.5v Vout for this circuit is 150v-225v (intended 170v)"
- note removed: "Connect later"
- note removed: "JLC Part U262-161N-4BVC11"
- note removed: "Mounting"
- note removed: "Package_SO:SOIC-8_3.9x4.9mm_P1.27mm"
- note removed: "Use ±1% feedback resistors to achieve an overall output voltage accuracy of ±5%"
- note removed: "Vout = Vref((R2 / R1) + 1) Vref = 1.5v Vout for this circuit is 150v-225v"
- moved on the sheet: BT1, C7, C8, R1, R2, R3, SW1, SW2, SW3, U3
