File: power_supply/power_supply.kicad_sch (KiCad schematic)
At the start: 20 parts, among them J2 Conn_01x10_Pin, J3 Conn_01x10_Pin, Q1 IRF644PBF, U1 MAX1771ESA+T

Commit message: Changed connectors
Changed connector from mcu to power supply to idc.
All switches now use a straight pinheader, with no pullups (now using
mcu pulldowns).
Parts:
- J2: footprint Connector_PinHeader_2.54mm:PinHeader_1x10_P2.54mm_Vertical -> Connector_IDC:IDC-Header_2x05_P2.54mm_Vertical
Changed lines of the file:
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@@
 	(title_block
 		(title "Power Supply Schematic")
-		(date "2024-05-29")
-		(rev "0.1.0")
+		(date "2024-06-06")
+		(rev "0.1.1")
 	)
 	(junction
@@
 			)
 		)
-		(property "Footprint" "Connector_PinHeader_2.54mm:PinHeader_1x10_P2.54mm_Vertical"
+		(property "Footprint" "Connector_IDC:IDC-Header_2x05_P2.54mm_Vertical"
 			(at 177.8 63.5 0)
 			(effects
